Commit message: Update hamo bot model

File: src/packages/linorobot2/linorobot2_description/urdf/robots/x2.urdf.xacro (robot description, xacro)
@@ -21,4 +21,15 @@
 <!-- Wheels -->
 <link name="front_left_wheel">
+    <inertial>
+    <mass value="1.0"/>
+    <origin xyz="0 0 0"/>
+    <inertia
+      ixx="0.001"
+      iyy="0.001"
+      izz="0.001"
+      ixy="0"
+      ixz="0"
+      iyz="0"/>
+  </inertial>
   <visual>
     <geometry>
@@ -28,4 +39,15 @@
 </link>
 <link name="front_right_wheel">
+    <inertial>
+    <mass value="1.0"/>
+    <origin xyz="0 0 0"/>
+    <inertia
+      ixx="0.001"
+      iyy="0.001"
+      izz="0.001"
+      ixy="0"
+      ixz="0"
+      iyz="0"/>
+  </inertial>
   <visual>
     <geometry>
@@ -35,4 +57,15 @@
 </link>
 <link name="rear_left_wheel">
+    <inertial>
+    <mass value="1.0"/>
+    <origin xyz="0 0 0"/>
+    <inertia
+      ixx="0.001"
+      iyy="0.001"
+      izz="0.001"
+      ixy="0"
+      ixz="0"
+      iyz="0"/>
+  </inertial>
   <visual>
     <geometry>
@@ -42,4 +75,15 @@
 </link>
 <link name="rear_right_wheel">
+    <inertial>
+    <mass value="1.0"/>
+    <origin xyz="0 0 0"/>
+    <inertia
+      ixx="0.001"
+      iyy="0.001"
+      izz="0.001"
+      ixy="0"
+      ixz="0"
+      iyz="0"/>
+  </inertial>
   <visual>
     <geometry>
