Commit message: Added camera

File: src/packages/linorobot2/linorobot2_description/urdf/robots/hamo_bot.urdf.xacro (robot description, xacro)
@@ -137,4 +137,52 @@
     <xacro:insert_block name="depth_sensor_pose" />
   </xacro:depth_sensor>
+  <!-- ================= REAR RGB CAMERA ================= -->
+  <link name="rear_camera_link">
+    <visual>
+      <geometry><box size="0.025 0.09 0.025"/></geometry>
+      <material name="black"><color rgba="0 0 0 1"/></material>
+    </visual>
+    <inertial>
+      <mass value="0.05"/>
+      <inertia ixx="1e-5" ixy="0" ixz="0" iyy="1e-5" iyz="0" izz="1e-5"/>
+    </inertial>
+  </link>
+  <joint name="rear_camera_joint" type="fixed">
+    <parent link="base_link"/>
+    <child link="rear_camera_link"/>
+    <!-- back face centre, mid height of base_link (origin at centre) -->
+    <origin xyz="${-base_length/2} 0 0" rpy="0 0 ${pi}"/>
+  </joint>
+  <link name="rear_camera_optical_frame"/>
+  <joint name="rear_camera_optical_joint" type="fixed">
+    <parent link="rear_camera_link"/>
+    <child link="rear_camera_optical_frame"/>
+    <origin xyz="0 0 0" rpy="${-pi/2} 0 ${-pi/2}"/>
+  </joint>
+  <gazebo reference="rear_camera_link">
+    <sensor name="rear_camera" type="camera">
+      <always_on>true</always_on>
+      <update_rate>30</update_rate>
+      <topic>rear_camera/image_raw</topic>
+      <gz_frame_id>rear_camera_optical_frame</gz_frame_id>
+      <camera>
+        <horizontal_fov>1.047</horizontal_fov>
+        <image>
+          <width>640</width>
+          <height>480</height>
+          <format>RGB_INT8</format>
+        </image>
+        <clip>
+          <near>0.1</near>
+          <far>50.0</far>
+        </clip>
+        <noise>
+          <type>gaussian</type>
+          <mean>0</mean>
+          <stddev>0.007</stddev>
+        </noise>
+      </camera>
+    </sensor>
+  </gazebo>
   <!-- ================= CONTROLLER ================= -->
   <xacro:diff_drive_controller
